File: ihm-esp32-core.kicad_pcb (KiCad board)
At the start: 2 copper layers, 92.4 x 62.9 mm, 75 parts, among them J1 Screw_Terminal_01x04, J2 Screw_Terminal_01x07, J3 Barrel_Jack_Switch, J4 Screw_Terminal_01x04, J5 Screw_Terminal_01x03, Q1 BC848, Q2 BC848, Q3 BC848, SW1 SW_MEC_5G, SW2 SW_MEC_5G, U1 ESP32-WROOM-32, U10 AZ1117-3.3, U11 TLP-2631, U3 TLP-2631, U4 LTV-357T, U5 CRE1S0505SC, U6 MAX485E, U7 CH340E, U8 PCF8563T, U9 AZ1117-5.0, Y1 Crystal_Small, Y3 Crystal

Commit message: Preparando para a release v2.0
Parts:
- removed D1: LL4148, Diode_SMD:D_MiniMELF
- removed J5: Screw_Terminal_01x03, Library:KF128L-3.5-3P
- removed U8: PCF8563T, Package_SO:SOIC-8_3.9x4.9mm_P1.27mm
- added C22: 100nF, Capacitor_SMD:C_0805_2012Metric, B.Cu at (155.7, 97.9)
- added J6: Screw_Terminal_01x03, Library:KF128L-3.5-3P, F.Cu at (208.9, 78.1)
- added R1: 22R, Resistor_SMD:R_0805_2012Metric, F.Cu at (206.8, 71.2)
- added R25: 330R, Resistor_SMD:R_0805_2012Metric, B.Cu at (157.8, 98.0)
- added R3: 22R, Resistor_SMD:R_0805_2012Metric, F.Cu at (206.9, 66.9)
- added U2: DS1307Z+, Package_SO:SOIC-8_3.9x4.9mm_P1.27mm, F.Cu at (134.6, 65.3)
- C1, C2: value 10uF/10V -> 100nF; footprint Capacitor_SMD:CP_Elec_4x5.3 -> Capacitor_SMD:C_0805_2012Metric
- C11: value 10nF/10V -> 100nF; footprint Capacitor_SMD:CP_Elec_5x5.9 -> Capacitor_SMD:C_0805_2012Metric
- C13: value 10uF/10V -> 100nF; footprint Capacitor_SMD:CP_Elec_5x5.9 -> Capacitor_SMD:C_0805_2012Metric
- C3: moved to B.Cu
- C9: value 10uF/25V -> 47uF/16V; footprint Capacitor_SMD:CP_Elec_6.3x5.2 -> Capacitor_SMD:C_1210_3225Metric
- D2: value LL4148 -> 1N4448W; footprint Diode_SMD:D_MiniMELF -> Diode_SMD:D_SOD-123; moved to B.Cu
- J1, J4: footprint Connector_PinHeader_2.54mm:PinHeader_1x04_P2.54mm_Vertical -> Library:kk-2.54-4P
- J2: footprint Connector_PinHeader_2.54mm:PinHeader_1x07_P2.54mm_Vertical -> Library:kk-2.54-7P
- moved D2 40.1 mm to (157.4, 101.0)
- moved J2 7.51 mm to (161.3, 88.9), turned to 0 degrees
- moved C2 5.47 mm to (190.4, 66.4)
- moved C1 5.41 mm to (185.3, 66.4)
- moved C3 5.36 mm to (134.8, 87.8), turned to 0 degrees
- moved J1 5.04 mm to (124.5, 89.5), turned to -90 degrees
- moved J4 3.88 mm to (148.3, 74.3), turned to -90 degrees
- moved C6 2.06 mm to (183.2, 66.4)
- moved C7 1.82 mm to (192.4, 66.4)
- moved C18 1.80 mm to (129.7, 96.1), turned to 90 degrees
- moved C9 1.34 mm to (194.0, 98.6)
- moved R24 1.27 mm to (152.6, 109.3), turned to 0 degrees
- moved C11 1.24 mm to (184.5, 98.0)
- moved C13 1.22 mm to (175.7, 98.0)
- moved Q3 0.63 mm to (156.8, 110.2)
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Connections:
- BZ1 pad 1: 5V -> Net-(BZ1--)
- C1 pad 1: VCC-IC -> 5V
- C1 pad 2: GND1 -> GND
- C2 pad 1: 5V -> VCC-IC
- C2 pad 2: GND -> GND1
- C5 pad 1: Net-(D1-K) -> 3V3
- D2 pad 1: Net-(D1-K) -> Net-(BZ1--)
- D2 pad 2: 3V3 -> Net-(BZ1-+)
Routing:
- net Net-(D1-K): track 7.86 -> 0.00 mm
- net Net-(BT2-+): track 7.62 -> 14.4 mm, vias 1 -> 0
- net Net-(BZ1--): track 0.00 -> 6.39 mm
- net LED1: track 53.8 -> 59.8 mm
- net 5V: track 145.8 -> 140.0 mm, vias 6 -> 7
- net 3V3: track 171.4 -> 174.6 mm
- net Net-(J1-Pin_2): track 5.91 -> 8.69 mm, vias 0 -> 1
- net B: track 9.58 -> 12.3 mm, vias 0 -> 1
- net Net-(J1-Pin_3): track 5.39 -> 8.05 mm
- net Net-(D3-A2): track 16.9 -> 18.9 mm
- net Net-(D4-A2): track 20.3 -> 22.3 mm
- net A: track 9.20 -> 11.2 mm, vias 0 -> 1
- net Net-(Q3-B): track 4.36 -> 2.41 mm
- net LED2: track 61.1 -> 62.5 mm
- net SCL: track 47.9 -> 46.8 mm
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Other:
- board text added: "ESP32-CORE V2.0"
- board text added: "RX"
- board text added: "TX"
- board text removed: "ESP32-CORE V1.0"
