File: ihm-esp32-core.kicad_sch (KiCad schematic)
At the start: 75 parts, among them J1 Screw_Terminal_01x04, J2 Screw_Terminal_01x07, J3 Barrel_Jack_Switch, J4 Screw_Terminal_01x04, J5 Screw_Terminal_01x03, Q1 BC848, Q2 BC848, Q3 BC848, SW1 SW_MEC_5G, SW2 SW_MEC_5G, U1 ESP32-WROOM-32, U10 AZ1117-3.3, U11 TLP-2631, U3 TLP-2631, U4 LTV-357T, U5 CRE1S0505SC, U6 MAX485E, U7 CH340E, U8 PCF8563T, U9 AZ1117-5.0, Y1 Crystal_Small, Y3 Crystal

Commit message: Preparando para a release v2.0
Parts:
- removed C1, C2: 10uF/10V, Capacitor_SMD:CP_Elec_4x5.3, symbol Device:C_Polarized_US
- removed C11: 10nF/10V, Capacitor_SMD:CP_Elec_5x5.9, symbol Device:C_Polarized_US
- removed C13: 10uF/10V, Capacitor_SMD:CP_Elec_5x5.9, symbol Device:C_Polarized_US
- removed C9: 10uF/25V, Capacitor_SMD:CP_Elec_6.3x5.2, symbol Device:C_Polarized_US
- removed D1, D2: LL4148, Diode_SMD:D_MiniMELF, symbol Diode:LL4148
- removed J5: Screw_Terminal_01x03, Library:KF128L-3.5-3P, symbol Connector:Screw_Terminal_01x03
- removed U8: PCF8563T, Package_SO:SOIC-8_3.9x4.9mm_P1.27mm, symbol Timer_RTC:PCF8563T
- added C1, C11, C13, C2, C22: 100nF, Capacitor_SMD:C_0805_2012Metric, symbol Device:C
- added C9: 47uF/16V, Capacitor_SMD:C_1210_3225Metric, symbol Device:C
- added D2: 1N4448W, Diode_SMD:D_SOD-123, symbol Diode:1N4448W
- added J6: Screw_Terminal_01x03, Library:KF128L-3.5-3P, symbol Connector:Screw_Terminal_01x03
- added R1, R3: 22R, Resistor_SMD:R_0805_2012Metric, symbol Device:R
- added R25: 330R, Resistor_SMD:R_0805_2012Metric, symbol Device:R
- added U2: DS1307Z+, Package_SO:SOIC-8_3.9x4.9mm_P1.27mm, symbol Timer_RTC:DS1307Z+
- J1, J4: footprint Connector_PinHeader_2.54mm:PinHeader_1x04_P2.54mm_Vertical -> Library:kk-2.54-4P
- J2: footprint Connector_PinHeader_2.54mm:PinHeader_1x07_P2.54mm_Vertical -> Library:kk-2.54-7P
Connections:
- net 3V3: now also C5.1, C13.1, U2.8 (VCC)
- net 5V: now also C1.1, C11.1, R25.1; no longer BZ1.1 (-)
- net A: now also J6.2 (Pin_2)
- net B: now also J6.1 (Pin_1)
- net GND: now also C1.2, C11.2, C13.2, C22.2, C9.2, U2.4 (GND)
- net GND1: now also C2.2, J6.3 (Pin_3), R1.1, R3.1
- net SCL: now also U2.6 (SCL)
- net SDA: now also U2.5 (SDA)
- net VCC-IC: now also C2.1
- net at BZ1.2 (+), Q3.3 (C): now also D2.2 (A)
- net at C10.1, J3.1, U9.3 (VI): now also C9.1
- net at D4.2 (A2), R18.1, U6.7 (B): now also R3.2
- net at D3.2 (A2), R17.1, U6.6 (A): now also R1.2
- net at Y1.1: now also U2.2 (X2)
- net at Y1.2: now also U2.1 (X1)
- net at BT2.1 (+): now also U2.3 (VBAT)
- new net: BZ1.1 (-), C22.1, D2.1 (K), R25.2
Other:
- moved on the sheet: BT2, BZ1, C20, C21, C5, D3, D4, D5, D6, R16, R17, R18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
